Commit message: updates to amiga_description launch, changed controllers file name

File: amiga_description/urdf/amiga.urdf.xacro (robot description, xacro)
@@ -6,5 +6,5 @@
     <xacro:arg name="amiga_prefix" default="amiga_"/>
     <xacro:arg name="amiga_parent" default="world" />
-    <xacro:arg name="mesh_base_path" default=""/>
+    <xacro:arg name="sim_gazebo" default="false"/>
     <!-- amiga macro -->
     <xacro:include filename="./amiga_macro.urdf.xacro" />
@@ -12,5 +12,5 @@
         amiga_prefix="$(arg amiga_prefix)"
         amiga_parent="$(arg amiga_parent)"
-        mesh_base_path="$(arg mesh_base_path)"
+        sim_gazebo="$(arg sim_gazebo)"
     />
     <!-- <joint name="world__$(arg amiga_prefix)base" type="fixed">

File: amiga_description/urdf/amiga_body.urdf.xacro (robot description, xacro)
@@ -1,5 +1,5 @@
 <?xml version="1.0"?>
 <robot xmlns:xacro="https://ros.org/wiki/xacro" name="amiga">
-  <xacro:macro name="amiga_body" params="prefix:='amiga_' amiga_parent:='world'">
+  <xacro:macro name="amiga_body" params="prefix:='amiga' amiga_parent:='world'">
     <material name="LightLightGrey">
       <color rgba="0.941 0.941 0.941 1.0"/>
@@ -19,9 +19,9 @@
     <!-- <xacro:property name="amiga_tool0_mount_position" value="-0.12825037 0.323256 0.99810607"/> -->
     <xacro:property name="amiga_tool0_mount_position" value="-0.225 0.323256 ${0.99810607+0.1}"/>
-    <link name="${prefix}body">
+    <link name="${prefix}__body">
       <visual>
         <origin rpy="0.0 0.0 0.0" xyz="0.0 0.0 0.0"/>
         <geometry>
-          <mesh filename="package://amiga_description/meshes/frame_on_amiga_v2_simplified.stl"/>
+          <mesh filename="file://$(find amiga_description)/meshes/frame_on_amiga_v2_simplified.stl"/>
         </geometry>
         <material name="LightLightGrey"/>
@@ -57,5 +57,5 @@
       </inertial>
     </link>
-    <link name="${prefix}tool0"/>
+    <link name="${prefix}__tool0"/>
     <!-- ================== -->
     <!--       Joints       -->
@@ -66,13 +66,13 @@
         <child link="${prefix}base"/>
     </joint> -->
-    <joint name="${prefix}base__${prefix}body" type="fixed">
+    <joint name="${prefix}__base--${prefix}__body" type="fixed">
         <origin rpy="0 0 0" xyz="0 0 0"/>
-        <parent link="${prefix}base"/>
-        <child link="${prefix}body"/>
+        <parent link="${prefix}__base"/>
+        <child link="${prefix}__body"/>
     </joint>
-    <joint name="${prefix}body--${prefix}tool0" type="fixed">
+    <joint name="${prefix}__body--${prefix}__tool0" type="fixed">
         <origin rpy="${amiga_tool0_mount_rotation}" xyz="${amiga_tool0_mount_position}"/>
-        <parent link="${prefix}body"/>
-        <child link="${prefix}tool0"/>
+        <parent link="${prefix}__body"/>
+        <child link="${prefix}__tool0"/>
     </joint>
   </xacro:macro>

File: amiga_description/urdf/amiga_macro.urdf.xacro (robot description, xacro)
@@ -1,5 +1,5 @@
 <?xml version="1.0"?>
 <robot xmlns:xacro="https://ros.org/wiki/xacro" name="amiga">
-<xacro:macro name="amiga_macro" params="amiga_prefix:='amiga_' amiga_parent:='world' mesh_base_path">
+<xacro:macro name="amiga_macro" params="amiga_prefix:='amiga_' amiga_parent:='world' sim_gazebo:='false'">
   <!-- ================== -->
   <!--     Amiga Macro    -->
@@ -11,58 +11,58 @@
   <!--       Links        -->
   <!-- ================== -->
-  <link name="${amiga_prefix}base"/>
+  <link name="${amiga_prefix}__base"/>
   <xacro:amiga_body
     prefix="${amiga_prefix}"
     amiga_parent="${amiga_prefix}base"
   />
-    <xacro:wheel
-        prefix="${amiga_prefix}"
-        wheel_name="left_wheel_front"
-        parent_link="${amiga_prefix}base"
-        joint_origin_xyz="0.344 0.5 0.22"
-        joint_origin_rpy="0 0 0"
-        joint_axis_xyz="0 1 0"
-        wheel_radius="0.25"
-        wheel_width="0.10"
-        wheel_mass="1.0"
-    />
-    <xacro:wheel
-        prefix="${amiga_prefix}"
-        wheel_name="right_wheel_front"
-        parent_link="${amiga_prefix}base"
-        joint_origin_xyz="0.344 -0.5 0.22"
-        joint_origin_rpy="0 0 0"
-        joint_axis_xyz="0 1 0"
-        wheel_radius="0.25"
-        wheel_width="0.10"
-        wheel_mass="1.0"
-    />
-    <xacro:wheel
-        prefix="${amiga_prefix}"
-        wheel_name="left_wheel_rear"
-        parent_link="${amiga_prefix}base"
-        joint_origin_xyz="-0.344 0.5 0.22"
-        joint_origin_rpy="0 0 0"
-        joint_axis_xyz="0 1 0"
-        wheel_radius="0.25"
-        wheel_width="0.10"
-        wheel_mass="1.0"
-    />
-    <xacro:wheel
-        prefix="${amiga_prefix}"
-        wheel_name="right_wheel_rear"
-        parent_link="${amiga_prefix}base"
-        joint_origin_xyz="-0.344 -0.5 0.22"
-        joint_origin_rpy="0 0 0"
-        joint_axis_xyz="0 1 0"
-        wheel_radius="0.25"
-        wheel_width="0.10"
-        wheel_mass="1.0"
-    />
-    <xacro:linear_slider_ros2_control
-        name="amiga"
-        prefix="${amiga_prefix}"
-        sim_gazebo="true"
-    />
+  <xacro:wheel
+    prefix="${amiga_prefix}"
+    wheel_name="left_wheel_front"
+    parent_link="${amiga_prefix}__base"
+    joint_origin_xyz="0.344 0.5 0.22"
+    joint_origin_rpy="0 0 0"
+    joint_axis_xyz="0 1 0"
+    wheel_radius="0.25"
+    wheel_width="0.10"
+    wheel_mass="1.0"
+  />
+  <xacro:wheel
+    prefix="${amiga_prefix}"
+    wheel_name="right_wheel_front"
+    parent_link="${amiga_prefix}__base"
+    joint_origin_xyz="0.344 -0.5 0.22"
+    joint_origin_rpy="0 0 0"
+    joint_axis_xyz="0 1 0"
+    wheel_radius="0.25"
+    wheel_width="0.10"
+    wheel_mass="1.0"
+  />
+  <xacro:wheel
+    prefix="${amiga_prefix}"
+    wheel_name="left_wheel_rear"
+    parent_link="${amiga_prefix}__base"
+    joint_origin_xyz="-0.344 0.5 0.22"
+    joint_origin_rpy="0 0 0"
+    joint_axis_xyz="0 1 0"
+    wheel_radius="0.25"
+    wheel_width="0.10"
+    wheel_mass="1.0"
+  />
+  <xacro:wheel
+    prefix="${amiga_prefix}"
+    wheel_name="right_wheel_rear"
+    parent_link="${amiga_prefix}__base"
+    joint_origin_xyz="-0.344 -0.5 0.22"
+    joint_origin_rpy="0 0 0"
+    joint_axis_xyz="0 1 0"
+    wheel_radius="0.25"
+    wheel_width="0.10"
+    wheel_mass="1.0"
+  />
+  <xacro:amiga_ros2_control
+    name="amiga"
+    prefix="${amiga_prefix}"
+    sim_gazebo="${sim_gazebo}"
+  />
 </xacro:macro>
 </robot>

File: amiga_description/urdf/amiga_ros2_control.urdf.xacro (robot description, xacro)
@@ -1,5 +1,5 @@
 <?xml version="1.0"?>
 <robot xmlns:xacro="http://www.ros.org/wiki/xacro">
-  <xacro:macro name="linear_slider_ros2_control" params="
+  <xacro:macro name="amiga_ros2_control" params="
       name
       prefix
@@ -11,5 +11,5 @@
     <!--    ros2_control    -->
     <!-- ================== -->
-    <ros2_control name="${name}_ros2_control" type="system">
+    <ros2_control name="amiga_ros2_control" type="system">
       <hardware>
         <xacro:if value="${use_mock_hardware}">
@@ -24,5 +24,5 @@
         </xacro:unless>
       </hardware>
-      <joint name="${prefix}left_wheel_front_joint">
+      <joint name="${prefix}__left_wheel_front_joint">
         <command_interface name="velocity"/>
         <state_interface name="velocity"/>
@@ -30,5 +30,5 @@
         <state_interface name="effort"/>
       </joint>
-      <joint name="${prefix}right_wheel_front_joint">
+      <joint name="${prefix}__right_wheel_front_joint">
         <command_interface name="velocity"/>
         <state_interface name="velocity"/>
@@ -36,5 +36,5 @@
         <state_interface name="effort"/>
       </joint>
-      <joint name="${prefix}left_wheel_rear_joint">
+      <joint name="${prefix}__left_wheel_rear_joint">
         <command_interface name="velocity"/>
         <state_interface name="velocity"/>
@@ -42,5 +42,5 @@
         <state_interface name="effort"/>
       </joint>
-      <joint name="${prefix}right_wheel_rear_joint">
+      <joint name="${prefix}__right_wheel_rear_joint">
         <command_interface name="velocity"/>
         <state_interface name="velocity"/>
@@ -52,5 +52,5 @@
     <plugin name="gz_ros2_control::GazeboSimROS2ControlPlugin"
             filename="libgz_ros2_control-system">
-      <parameters>$(find amiga_description)/config/diff_drive_controller.yaml</parameters>
+      <parameters>$(find amiga_description)/config/amiga_controllers.yaml</parameters>
       <controller_manager_name>controller_manager</controller_manager_name>
     </plugin>

File: amiga_description/urdf/amiga_wheel.urdf.xacro (robot description, xacro)
@@ -3,5 +3,5 @@
   <xacro:macro name="wheel"
     params="prefix wheel_name parent_link joint_origin_xyz joint_origin_rpy joint_axis_xyz wheel_radius wheel_width wheel_mass">
-    <link name="${prefix}${wheel_name}">
+    <link name="${prefix}__${wheel_name}">
       <visual>
         <origin xyz="0 0 0" rpy="1.5708 0 0"/>
@@ -26,8 +26,8 @@
       </inertial>
     </link>
-    <joint name="${prefix}${wheel_name}_joint" type="continuous">
+    <joint name="${prefix}__${wheel_name}_joint" type="continuous">
       <origin xyz="${joint_origin_xyz}" rpy="${joint_origin_rpy}"/>
       <parent link="${parent_link}"/>
-      <child link="${prefix}${wheel_name}"/>
+      <child link="${prefix}__${wheel_name}"/>
       <axis xyz="${joint_axis_xyz}"/>
       <limit effort="30.0" velocity="50.0"/>

Commit message: fixed rebase errors

File: amiga_description/urdf/amiga.urdf.xacro (robot description, xacro)
@@ -4,7 +4,7 @@
     <link name="world" />
     <!-- Args -->
-    <xacro:arg name="amiga_prefix" default="amiga__"/>
+    <xacro:arg name="amiga_prefix" default="amiga"/>
     <xacro:arg name="amiga_parent" default="world" />
-    <xacro:arg name="mesh_base_path" default=""/>
+    <xacro:arg name="sim_gazebo" default="false"/>
     <!-- amiga macro -->
     <xacro:include filename="./amiga_macro.urdf.xacro" />
@@ -12,10 +12,5 @@
         amiga_prefix="$(arg amiga_prefix)"
         amiga_parent="$(arg amiga_parent)"
-        mesh_base_path="$(arg mesh_base_path)"
+        sim_gazebo="$(arg sim_gazebo)"
     />
-    <joint name="world__$(arg amiga_prefix)base" type="fixed">
-        <origin xyz="0.0 0.0 0.0" rpy="0 0 0"/>
-        <parent link="world" />
-        <child link="$(arg amiga_prefix)base" />
-    </joint>
 </robot>

File: amiga_description/urdf/amiga_body.urdf.xacro (robot description, xacro)
@@ -1,5 +1,5 @@
 <?xml version="1.0"?>
 <robot xmlns:xacro="https://ros.org/wiki/xacro" name="amiga">
-  <xacro:macro name="amiga_body" params="prefix:='amiga__' amiga_parent:='world'">
+  <xacro:macro name="amiga_body" params="prefix:='amiga' amiga_parent:='world'">
     <material name="LightLightGrey">
       <color rgba="0.941 0.941 0.941 1.0"/>
@@ -19,5 +19,5 @@
     <!-- <xacro:property name="amiga_tool0_mount_position" value="-0.12825037 0.323256 0.99810607"/> -->
     <xacro:property name="amiga_tool0_mount_position" value="-0.225 0.323256 ${0.99810607+0.1}"/>
-    <link name="${prefix}body">
+    <link name="${prefix}__body">
       <visual>
         <origin rpy="0.0 0.0 0.0" xyz="0.0 0.0 0.0"/>
@@ -27,22 +27,22 @@
         <material name="LightLightGrey"/>
       </visual>
-      <collision>
+      <!-- <collision>
         <origin rpy="0.0 0.0 0.0" xyz="0.0 0.0 ${amiga_collision_box0_z / 2}"/>
         <geometry>
           <box size="${amiga_collision_box0_x} ${amiga_collision_box0_y} ${amiga_collision_box0_z}"/>
         </geometry>
-      </collision>
-      <collision>
+      </collision> -->
+      <!-- <collision>
         <origin rpy="0.0 0.0 0.0" xyz="0.0 -${amiga_collision_box1_y / 5} ${amiga_collision_box0_z}" />
         <geometry>
           <box size="${amiga_collision_box1_x} ${amiga_collision_box1_y} ${amiga_collision_box1_z}" />
         </geometry>
-      </collision>
-      <collision>
+      </collision> -->
+      <!-- <collision>
         <origin rpy="0.0 0.0 0.0" xyz="${amiga_collision_box0_x / 2 - amiga_collision_box2_x / 2} ${amiga_collision_box2_y / 3} ${amiga_collision_box0_z + amiga_collision_box1_z}" />
         <geometry>
           <box size="${amiga_collision_box2_x} ${amiga_collision_box2_y} ${amiga_collision_box2_z}" />
         </geometry>
-      </collision>
+      </collision> -->
       <inertial>
         <origin rpy="0 0 0" xyz="0.0 0.0 0.0"/>
@@ -57,22 +57,17 @@
       </inertial>
     </link>
-    <link name="${prefix}tool0"/>
+    <link name="${prefix}__tool0"/>
     <!-- ================== -->
     <!--       Joints       -->
     <!-- ================== -->
-    <joint name="${amiga_parent}--${prefix}base" type ="fixed">
+    <joint name="${prefix}__base--${prefix}__body" type="fixed">
         <origin rpy="0 0 0" xyz="0 0 0"/>
-        <parent link="${amiga_parent}"/>
-        <child link="${prefix}base"/>
+        <parent link="${prefix}__base"/>
+        <child link="${prefix}__body"/>
     </joint>
-    <joint name="${prefix}base--${prefix}body" type="fixed">
-        <origin rpy="0 0 0" xyz="0 0 0"/>
-        <parent link="${prefix}base"/>
-        <child link="${prefix}body"/>
-    </joint>
-    <joint name="${prefix}body--${prefix}tool0" type="fixed">
+    <joint name="${prefix}__body--${prefix}__tool0" type="fixed">
         <origin rpy="${amiga_tool0_mount_rotation}" xyz="${amiga_tool0_mount_position}"/>
-        <parent link="${prefix}body"/>
-        <child link="${prefix}tool0"/>
+        <parent link="${prefix}__body"/>
+        <child link="${prefix}__tool0"/>
     </joint>
   </xacro:macro>

File: amiga_description/urdf/amiga_macro.urdf.xacro (robot description, xacro)
@@ -1,5 +1,5 @@
 <?xml version="1.0"?>
 <robot xmlns:xacro="https://ros.org/wiki/xacro" name="amiga">
-<xacro:macro name="amiga_macro" params="amiga_prefix:='amiga__' amiga_parent:='world' mesh_base_path">
+<xacro:macro name="amiga_macro" params="amiga_prefix:='amiga_' amiga_parent:='world' sim_gazebo:='false'">
   <!-- ================== -->
   <!--     Amiga Macro    -->
@@ -7,44 +7,62 @@
   <xacro:include filename="./amiga_body.urdf.xacro" />
   <xacro:include filename="./amiga_wheel.urdf.xacro" />
+  <xacro:include filename="./amiga_ros2_control.urdf.xacro" />
   <!-- ================== -->
   <!--       Links        -->
   <!-- ================== -->
-  <link name="${amiga_prefix}base"/>
+  <link name="${amiga_prefix}__base"/>
   <xacro:amiga_body
     prefix="${amiga_prefix}"
     amiga_parent="${amiga_prefix}base"
   />
-    <xacro:wheel
-        prefix="${amiga_prefix}"
-        wheel_name="left_wheel_front"
-        parent_link="base"
-        joint_origin_xyz="0.4 0.25 0.05"
-        joint_origin_rpy="0 0 0"
-        joint_axis_xyz="0 1 0"
-    />
-    <xacro:wheel
-        prefix="${amiga_prefix}"
-        wheel_name="right_wheel_front"
-        parent_link="base"
-        joint_origin_xyz="0.4 -0.25 0.05"
-        joint_origin_rpy="0 0 0"
-        joint_axis_xyz="0 1 0"
-    />
-    <xacro:wheel
-        prefix="${amiga_prefix}"
-        wheel_name="left_wheel_rear"
-        parent_link="base"
-        joint_origin_xyz="-0.4 0.25 0.05"
-        joint_origin_rpy="0 0 0"
-        joint_axis_xyz="0 1 0"
-    />
-    <xacro:wheel
-        prefix="${amiga_prefix}"
-        wheel_name="right_wheel_rear"
-        parent_link="base"
-        joint_origin_xyz="-0.4 -0.25 0.05"
-        joint_origin_rpy="0 0 0"
-        joint_axis_xyz="0 1 0"
-    />
+  <xacro:wheel
+    prefix="${amiga_prefix}"
+    wheel_name="left_wheel_front"
+    parent_link="${amiga_prefix}__base"
+    joint_origin_xyz="0.344 0.5 0.22"
+    joint_origin_rpy="0 0 0"
+    joint_axis_xyz="0 1 0"
+    wheel_radius="0.25"
+    wheel_width="0.10"
+    wheel_mass="1.0"
+  />
+  <xacro:wheel
+    prefix="${amiga_prefix}"
+    wheel_name="right_wheel_front"
+    parent_link="${amiga_prefix}__base"
+    joint_origin_xyz="0.344 -0.5 0.22"
+    joint_origin_rpy="0 0 0"
+    joint_axis_xyz="0 1 0"
+    wheel_radius="0.25"
+    wheel_width="0.10"
+    wheel_mass="1.0"
+  />
+  <xacro:wheel
+    prefix="${amiga_prefix}"
+    wheel_name="left_wheel_rear"
+    parent_link="${amiga_prefix}__base"
+    joint_origin_xyz="-0.344 0.5 0.22"
+    joint_origin_rpy="0 0 0"
+    joint_axis_xyz="0 1 0"
+    wheel_radius="0.25"
+    wheel_width="0.10"
+    wheel_mass="1.0"
+  />
+  <xacro:wheel
+    prefix="${amiga_prefix}"
+    wheel_name="right_wheel_rear"
+    parent_link="${amiga_prefix}__base"
+    joint_origin_xyz="-0.344 -0.5 0.22"
+    joint_origin_rpy="0 0 0"
+    joint_axis_xyz="0 1 0"
+    wheel_radius="0.25"
+    wheel_width="0.10"
+    wheel_mass="1.0"
+  />
+  <xacro:amiga_ros2_control
+    name="amiga"
+    prefix="${amiga_prefix}"
+    sim_gazebo="${sim_gazebo}"
+  />
 </xacro:macro>
 </robot>

File: amiga_description/urdf/amiga_ros2_control.urdf.xacro (robot description, xacro)
@@ -1,5 +1,5 @@
 <?xml version="1.0"?>
 <robot xmlns:xacro="http://www.ros.org/wiki/xacro">
-  <xacro:macro name="linear_slider_ros2_control" params="
+  <xacro:macro name="amiga_ros2_control" params="
       name
       prefix
@@ -11,5 +11,5 @@
     <!--    ros2_control    -->
     <!-- ================== -->
-    <ros2_control name="${name}_ros2_control" type="system">
+    <ros2_control name="amiga_ros2_control" type="system">
       <hardware>
         <xacro:if value="${use_mock_hardware}">
@@ -18,5 +18,5 @@
         </xacro:if>
         <xacro:if value="${sim_gazebo}">
-          <plugin>gazebo_ros2_control/GazeboSystem</plugin>
+          <plugin>gz_ros2_control/GazeboSimSystem</plugin>
         </xacro:if>
         <xacro:unless value="${use_mock_hardware or sim_gazebo}">
@@ -50,6 +50,8 @@
     </ros2_control>
     <gazebo>
-      <plugin filename="libgazebo_ros2_control.so" name="gazebo_ros2_control">
-        <parameters>$(find amiga_description)/config/diff_drive_controller.yaml</parameters>
+      <plugin name="gz_ros2_control::GazeboSimROS2ControlPlugin"
+              filename="libgz_ros2_control-system">
+        <parameters>$(find amiga_description)/config/amiga_controllers.yaml</parameters>
+        <controller_manager_name>controller_manager</controller_manager_name>
       </plugin>
     </gazebo>

File: amiga_description/urdf/amiga_wheel.urdf.xacro (robot description, xacro)
@@ -1,12 +1,40 @@
 <?xml version="1.0"?>
 <robot xmlns:xacro="http://ros.org/wiki/xacro">
-  <xacro:macro name="wheel" params="prefix wheel_name parent_link joint_origin_xyz joint_origin_rpy joint_axis_xyz">
-    <link name="${prefix}__${wheel_name}"/>
+  <xacro:macro name="wheel"
+    params="prefix wheel_name parent_link joint_origin_xyz joint_origin_rpy joint_axis_xyz wheel_radius wheel_width wheel_mass">
+    <link name="${prefix}__${wheel_name}">
+      <visual>
+        <origin xyz="0 0 0" rpy="1.5708 0 0"/>
+        <geometry>
+          <cylinder radius="${wheel_radius}" length="${wheel_width}"/>
+        </geometry>
+      </visual>
+      <collision>
+        <origin xyz="0 0 0" rpy="1.5708 0 0"/>
+        <geometry>
+          <cylinder radius="${wheel_radius}" length="${wheel_width}"/>
+        </geometry>
+      </collision>
+      <inertial>
+        <origin xyz="0 0 0" rpy="1.5708 0 0"/>
+        <mass value="${wheel_mass}"/>
+        <inertia
+          ixx="${(wheel_mass*(3*wheel_radius*wheel_radius + wheel_width*wheel_width))/12.0}"
+          iyy="${(wheel_mass*wheel_radius*wheel_radius)/2.0}"
+          izz="${(wheel_mass*(3*wheel_radius*wheel_radius + wheel_width*wheel_width))/12.0}"
+          ixy="0" ixz="0" iyz="0"/>
+      </inertial>
+    </link>
     <joint name="${prefix}__${wheel_name}_joint" type="continuous">
       <origin xyz="${joint_origin_xyz}" rpy="${joint_origin_rpy}"/>
-      <parent link="${prefix}__${parent_link}"/>
+      <parent link="${parent_link}"/>
       <child link="${prefix}__${wheel_name}"/>
       <axis xyz="${joint_axis_xyz}"/>
+      <limit effort="30.0" velocity="50.0"/>
+      <dynamics damping="0.1" friction="0.1"/>
     </joint>
+    <gazebo reference="${prefix}__${wheel_name}_joint">
+      <preserveFixedJoint>false</preserveFixedJoint>
+    </gazebo>
   </xacro:macro>
 </robot>

Commit message: small fixes to urdf __

File: amiga_description/urdf/amiga.urdf.xacro (robot description, xacro)
@@ -2,5 +2,5 @@
 <robot xmlns:xacro="https://ros.org/wiki/xacro" name="amiga">
     <!-- World link -->
-    <link name="world" />
+    <!-- <link name="world" /> -->
     <!-- Args -->
     <xacro:arg name="amiga_prefix" default="amiga"/>

File: amiga_description/urdf/amiga_macro.urdf.xacro (robot description, xacro)
@@ -14,5 +14,5 @@
   <xacro:amiga_body
     prefix="${amiga_prefix}"
-    amiga_parent="${amiga_prefix}base"
+    amiga_parent="${amiga_prefix}__base"
   />
   <xacro:wheel
