Commit message: tried debugging movement, no luck yet

File: amiga_description/urdf/amiga_macro.urdf.xacro (robot description, xacro)
@@ -1,11 +1,15 @@
 <?xml version="1.0"?>
 <robot xmlns:xacro="https://ros.org/wiki/xacro" name="amiga">
-<xacro:macro name="amiga_macro" params="amiga_prefix:='amiga_' amiga_parent:='world' sim_gazebo:='false'">
+<xacro:macro name="amiga_macro" params="amiga_prefix:='amiga' amiga_parent:='world' sim_gazebo:='false'">
   <!-- ================== -->
   <!--     Amiga Macro    -->
   <!-- ================== -->
   <xacro:include filename="./amiga_body.urdf.xacro" />
+  <xacro:include filename="./amiga_lidar.urdf.xacro" />
   <xacro:include filename="./amiga_wheel.urdf.xacro" />
   <xacro:include filename="./amiga_ros2_control.urdf.xacro" />
+  <xacro:property name="wheel_radius" value="0.25"/>
+  <xacro:property name="wheel_width" value="0.10"/>
+  <xacro:property name="wheel_mass" value="1.0"/>
   <!-- ================== -->
   <!--       Links        -->
@@ -16,4 +20,9 @@
     amiga_parent="${amiga_prefix}__base"
   />
+  <xacro:lidar
+    prefix="${amiga_prefix}"
+    lidar_name="lidar"
+    parent_link="${amiga_prefix}__base"
+  />
   <xacro:wheel
     prefix="${amiga_prefix}"
@@ -23,7 +32,7 @@
     joint_origin_rpy="0 0 0"
     joint_axis_xyz="0 1 0"
-    wheel_radius="0.25"
-    wheel_width="0.10"
-    wheel_mass="1.0"
+    wheel_radius="${wheel_radius}"
+    wheel_width="${wheel_width}"
+    wheel_mass="${wheel_mass}"
   />
   <xacro:wheel
@@ -34,7 +43,7 @@
     joint_origin_rpy="0 0 0"
     joint_axis_xyz="0 1 0"
-    wheel_radius="0.25"
-    wheel_width="0.10"
-    wheel_mass="1.0"
+    wheel_radius="${wheel_radius}"
+    wheel_width="${wheel_width}"
+    wheel_mass="${wheel_mass}"
   />
   <xacro:wheel
@@ -45,7 +54,7 @@
     joint_origin_rpy="0 0 0"
     joint_axis_xyz="0 1 0"
-    wheel_radius="0.25"
-    wheel_width="0.10"
-    wheel_mass="1.0"
+    wheel_radius="${wheel_radius}"
+    wheel_width="${wheel_width}"
+    wheel_mass="${wheel_mass}"
   />
   <xacro:wheel
@@ -56,7 +65,7 @@
     joint_origin_rpy="0 0 0"
     joint_axis_xyz="0 1 0"
-    wheel_radius="0.25"
-    wheel_width="0.10"
-    wheel_mass="1.0"
+    wheel_radius="${wheel_radius}"
+    wheel_width="${wheel_width}"
+    wheel_mass="${wheel_mass}"
   />
   <xacro:amiga_ros2_control

File: amiga_description/urdf/amiga_ros2_control.urdf.xacro (robot description, xacro)
@@ -54,4 +54,5 @@
         <parameters>$(find amiga_description)/config/amiga_controllers.yaml</parameters>
         <controller_manager_name>controller_manager</controller_manager_name>
+        <hold_joints>false</hold_joints>
       </plugin>
     </gazebo>

Commit message: messing around with diff drive parameters

File: amiga_description/urdf/amiga_macro.urdf.xacro (robot description, xacro)
@@ -33,9 +33,20 @@
   <xacro:wheel
     prefix="${amiga_prefix}"
-    wheel_name="left_wheel_front"
+    wheel_name="right_wheel_rear"
     parent_link="${amiga_prefix}__base"
     joint_origin_xyz="0.344 0.5 0.22"
     joint_origin_rpy="0 0 0"
-    joint_axis_xyz="0 1 0"
+    joint_axis_xyz="0 -1 0"
+    wheel_radius="${wheel_radius}"
+    wheel_width="${wheel_width}"
+    wheel_mass="${wheel_mass}"
+  />
+  <xacro:wheel
+    prefix="${amiga_prefix}"
+    wheel_name="left_wheel_rear"
+    parent_link="${amiga_prefix}__base"
+    joint_origin_xyz="0.344 -0.5 0.22"
+    joint_origin_rpy="0 0 0"
+    joint_axis_xyz="0 -1 0"
     wheel_radius="${wheel_radius}"
     wheel_width="${wheel_width}"
@@ -46,7 +57,7 @@
     wheel_name="right_wheel_front"
     parent_link="${amiga_prefix}__base"
-    joint_origin_xyz="0.344 -0.5 0.22"
+    joint_origin_xyz="-0.344 0.5 0.22"
     joint_origin_rpy="0 0 0"
-    joint_axis_xyz="0 1 0"
+    joint_axis_xyz="0 -1 0"
     wheel_radius="${wheel_radius}"
     wheel_width="${wheel_width}"
@@ -55,20 +66,9 @@
   <xacro:wheel
     prefix="${amiga_prefix}"
-    wheel_name="left_wheel_rear"
-    parent_link="${amiga_prefix}__base"
-    joint_origin_xyz="-0.344 0.5 0.22"
-    joint_origin_rpy="0 0 0"
-    joint_axis_xyz="0 1 0"
-    wheel_radius="${wheel_radius}"
-    wheel_width="${wheel_width}"
-    wheel_mass="${wheel_mass}"
-  />
-  <xacro:wheel
-    prefix="${amiga_prefix}"
-    wheel_name="right_wheel_rear"
+    wheel_name="left_wheel_front"
     parent_link="${amiga_prefix}__base"
     joint_origin_xyz="-0.344 -0.5 0.22"
     joint_origin_rpy="0 0 0"
-    joint_axis_xyz="0 1 0"
+    joint_axis_xyz="0 -1 0"
     wheel_radius="${wheel_radius}"
     wheel_width="${wheel_width}"

File: amiga_description/urdf/amiga_wheel.urdf.xacro (robot description, xacro)
@@ -17,10 +17,10 @@
       </collision>
       <inertial>
-        <origin xyz="0 0 0" rpy="1.5708 0 0"/>
+        <origin xyz="0 0 0" rpy="0 0 0"/>
         <mass value="${wheel_mass}"/>
         <inertia
-          ixx="${(wheel_mass*(3*wheel_radius*wheel_radius + wheel_width*wheel_width))/12.0}"
-          iyy="${(wheel_mass*wheel_radius*wheel_radius)/2.0}"
-          izz="${(wheel_mass*(3*wheel_radius*wheel_radius + wheel_width*wheel_width))/12.0}"
+          ixx="${(wheel_mass*(3*wheel_radius**2 + wheel_width**2))/12.0}"
+          iyy="${(wheel_mass*wheel_radius**2)/2.0}"
+          izz="${(wheel_mass*(3*wheel_radius**2 + wheel_width**2))/12.0}"
           ixy="0" ixz="0" iyz="0"/>
       </inertial>
@@ -32,8 +32,13 @@
       <axis xyz="${joint_axis_xyz}"/>
       <limit effort="30.0" velocity="50.0"/>
-      <dynamics damping="0.1" friction="0.1"/>
+      <dynamics damping="0.5" friction="0.5"/>
     </joint>
     <gazebo reference="${prefix}__${wheel_name}_joint">
-      <preserveFixedJoint>false</preserveFixedJoint>
+      <mu1>1.0</mu1> <!-- longitudinal friction (rolling direction) -->
+      <mu2>0.3</mu2> <!-- lateral friction (sideways direction) -->
+      <kp>1e6</kp>         <!-- contact stiffness -->
+      <kd>10.0</kd>        <!-- contact damping -->
+      <minDepth>0.001</minDepth> <!-- minimum depth for contact -->
+      <maxContacts>1</maxContacts>
     </gazebo>
   </xacro:macro>
