Commit message: updated lidar params

File: amiga_description/urdf/amiga_lidar.urdf.xacro (robot description, xacro)
@@ -4,4 +4,5 @@
     <xacro:property name="lidar_mass" value="1.0"/>
     <xacro:property name="lidar_xyz" value="-0.65 0 ${1.132/2}"/>
+    <xacro:property name="lidar_rpy" value="0 0 3.14159265359"/>
     <link name="${prefix}__${lidar_name}">
       <visual>
@@ -24,5 +25,5 @@
     </link>
     <joint name="${prefix}__${lidar_name}_joint" type="fixed">
-      <origin xyz="${lidar_xyz}" rpy="0 0 0"/>
+      <origin xyz="${lidar_xyz}" rpy="${lidar_rpy}"/>
       <parent link="${parent_link}"/>
       <child link="${prefix}__${lidar_name}"/>
@@ -41,6 +42,6 @@
               <samples>360</samples>
               <resolution>1</resolution>
-              <min_angle>-3.14159</min_angle>
-              <max_angle>3.14159</max_angle>
+              <min_angle>-1.57079632679</min_angle>
+              <max_angle>1.57079632679</max_angle>
             </horizontal>
           </scan>

Commit message: lowering lidar to test

File: amiga_description/urdf/amiga_lidar.urdf.xacro (robot description, xacro)
@@ -3,5 +3,5 @@
   <xacro:macro name="lidar" params="prefix lidar_name parent_link">
     <xacro:property name="lidar_mass" value="1.0"/>
-    <xacro:property name="lidar_xyz" value="-0.65 0 ${1.132/2}"/>
+    <xacro:property name="lidar_xyz" value="-0.65 0 ${0.132/2}"/>
     <link name="${prefix}__${lidar_name}">
       <visual>

Commit message: changed location of lidar, is detecting things well -- gotta add humble localization

File: amiga_description/urdf/amiga_lidar.urdf.xacro (robot description, xacro)
@@ -3,5 +3,5 @@
   <xacro:macro name="lidar" params="prefix lidar_name parent_link">
     <xacro:property name="lidar_mass" value="1.0"/>
-    <xacro:property name="lidar_xyz" value="-0.65 0 ${1.132/2}"/>
+    <xacro:property name="lidar_xyz" value="-0.65 0 ${0.232/2}"/>
     <xacro:property name="lidar_rpy" value="0 0 3.14159265359"/>
     <link name="${prefix}__${lidar_name}">

File: amiga_description/urdf/amiga_macro.urdf.xacro (robot description, xacro)
@@ -10,5 +10,5 @@
   <xacro:include filename="./amiga_wheel.urdf.xacro" />
   <xacro:include filename="./amiga_ros2_control.urdf.xacro" />
-  <xacro:property name="wheel_radius" value="0.25"/>
+  <xacro:property name="wheel_radius" value="0.2"/>
   <xacro:property name="wheel_width" value="0.10"/>
   <xacro:property name="wheel_mass" value="1.0"/>
