Commit message: adding imu, testing

File: amiga_description/urdf/amiga_imu.urdf.xacro (robot description, xacro)
@@ -1,84 +1,84 @@
 <?xml version="1.0"?>
 <robot xmlns:xacro="http://ros.org">
-  <xacro:macro name="imu" params="prefix imu_name parent_link">
-    <xacro:property name="imu_mass" value="0.1"/>
-    <xacro:property name="imu_xyz" value="0 0.1 0.8"/>
-    <xacro:property name="imu_rpy" value="0 0 0"/>
-    <link name="${prefix}__${imu_name}">
-      <visual>
-        <origin xyz="0 0 0" rpy="0 0 0"/>
-        <geometry>
-          <box size="0.05 0.05 0.02"/>
-        </geometry>
-      </visual>
-      <collision>
-        <origin xyz="0 0 0" rpy="0 0 0"/>
-        <geometry>
-          <box size="0.05 0.05 0.02"/>
-        </geometry>
-      </collision>
-      <inertial>
-        <origin xyz="0 0 0" rpy="0 0 0"/>
-        <mass value="0.1"/>
-        <inertia ixx="0.0001" iyy="0.0001" izz="0.0001" ixy="0" ixz="0" iyz="0"/>
-      </inertial>
-    </link>
-    <joint name="${prefix}__${imu_name}_joint" type="fixed">
-      <origin xyz="${imu_xyz}" rpy="${imu_rpy}"/>
-      <parent link="${parent_link}"/>
-      <child link="${prefix}__${imu_name}"/>
-    </joint>
-    <!-- Use the LINK name here, not the joint name -->
-    <gazebo reference="${prefix}__${imu_name}">
-      <sensor name="${prefix}__${imu_name}_sensor" type="imu">
-        <gz_frame_id>${prefix}__${imu_name}</gz_frame_id>
-        <topic>imu</topic>
-        <always_on>true</always_on>
-        <visualize>false</visualize>
-        <update_rate>100.0</update_rate>
-        <imu>
-          <angular_velocity>
-            <x>
-              <noise type="gaussian">
-                <mean>0.0</mean>
-                <stddev>0.009</stddev>
-              </noise>
-            </x>
-            <y>
-              <noise type="gaussian">
-                <mean>0.0</mean>
-                <stddev>0.009</stddev>
-              </noise>
-            </y>
-            <z>
-              <noise type="gaussian">
-                <mean>0.0</mean>
-                <stddev>0.009</stddev>
-              </noise>
-            </z>
-          </angular_velocity>
-          <linear_acceleration>
-            <x>
-              <noise type="gaussian">
-                <mean>0.0</mean>
-                <stddev>0.021</stddev>
-              </noise>
-            </x>
-            <y>
-              <noise type="gaussian">
-                <mean>0.0</mean>
-                <stddev>0.021</stddev>
-              </noise>
-            </y>
-            <z>
-              <noise type="gaussian">
-                <mean>0.0</mean>
-                <stddev>0.021</stddev>
-              </noise>
-            </z>
-          </linear_acceleration>
-        </imu>
-      </sensor>
-    </gazebo>
-  </xacro:macro>
+ <xacro:macro name="imu" params="prefix imu_name parent_link">
+   <xacro:property name="imu_mass" value="0.1"/>
+   <xacro:property name="imu_xyz" value="0 0.1 0.8"/>
+   <xacro:property name="imu_rpy" value="0 0 0"/>
+   <link name="${prefix}__${imu_name}">
+     <visual>
+       <origin xyz="0 0 0" rpy="0 0 0"/>
+       <geometry>
+         <box size="0.05 0.05 0.02"/>
+       </geometry>
+     </visual>
+     <collision>
+       <origin xyz="0 0 0" rpy="0 0 0"/>
+       <geometry>
+         <box size="0.05 0.05 0.02"/>
+       </geometry>
+     </collision>
+     <inertial>
+       <origin xyz="0 0 0" rpy="0 0 0"/>
+       <mass value="0.1"/>
+       <inertia ixx="0.0001" iyy="0.0001" izz="0.0001" ixy="0" ixz="0" iyz="0"/>
+     </inertial>
+   </link>
+   <joint name="${prefix}__${imu_name}_joint" type="fixed">
+     <origin xyz="${imu_xyz}" rpy="${imu_rpy}"/>
+     <parent link="${parent_link}"/>
+     <child link="${prefix}__${imu_name}"/>
+   </joint>
+   <!-- Use the LINK name here, not the joint name -->
+   <gazebo reference="${prefix}__${imu_name}">
+     <sensor name="${prefix}__${imu_name}_sensor" type="imu">
+       <gz_frame_id>${prefix}__${imu_name}</gz_frame_id>
+       <topic>imu</topic>
+       <always_on>true</always_on>
+       <visualize>false</visualize>
+       <update_rate>100.0</update_rate>
+       <imu>
+         <angular_velocity>
+           <x>
+             <noise type="gaussian">
+               <mean>0.0</mean>
+               <stddev>0.009</stddev>
+             </noise>
+           </x>
+           <y>
+             <noise type="gaussian">
+               <mean>0.0</mean>
+               <stddev>0.009</stddev>
+             </noise>
+           </y>
+           <z>
+             <noise type="gaussian">
+               <mean>0.0</mean>
+               <stddev>0.009</stddev>
+             </noise>
+           </z>
+         </angular_velocity>
+         <linear_acceleration>
+           <x>
+             <noise type="gaussian">
+               <mean>0.0</mean>
+               <stddev>0.021</stddev>
+             </noise>
+           </x>
+           <y>
+             <noise type="gaussian">
+               <mean>0.0</mean>
+               <stddev>0.021</stddev>
+             </noise>
+           </y>
+           <z>
+             <noise type="gaussian">
+               <mean>0.0</mean>
+               <stddev>0.021</stddev>
+             </noise>
+           </z>
+         </linear_acceleration>
+       </imu>
+     </sensor>
+   </gazebo>
+ </xacro:macro>
 </robot>
