Commit message: changed sensor configs to match real-world sensors

File: amiga_description/urdf/amiga_gps.urdf.xacro (robot description, xacro)
@@ -1,4 +1,4 @@
 <?xml version="1.0"?>
-<robot xmlns:xacro="http://www.ros.org">
+<robot xmlns:xacro="http://www.ros.org/wiki/xacro">
   <xacro:macro name="gps" params="prefix gps_name parent_link">
     <joint name="${prefix}__${gps_name}_joint" type="fixed">
@@ -17,4 +17,20 @@
         <update_rate>10</update_rate>
         <topic>gps/fix</topic>
+        <gps>
+          <position_sensing>
+            <horizontal>
+              <noise type="gaussian">
+                <mean>0.0</mean>
+                <stddev>0.000012631971681894632</stddev> <!-- 1m in degrees at lat=44.567774396988014 -->
+              </noise>
+            </horizontal>
+            <vertical>
+              <noise type="gaussian">
+                <mean>0.0</mean>
+                <stddev>10.0</stddev> <!-- meters for vertical position -->
+              </noise>
+            </vertical>
+          </position_sensing>
+        </gps>
       </sensor>
     </gazebo>

File: amiga_description/urdf/amiga_imu.urdf.xacro (robot description, xacro)
@@ -1,4 +1,4 @@
 <?xml version="1.0"?>
-<robot xmlns:xacro="http://ros.org">
+<robot xmlns:xacro="http://www.ros.org/wiki/xacro">
   <xacro:macro name="imu" params="prefix imu_name parent_link">
     <xacro:property name="imu_mass" value="0.1"/>
@@ -45,5 +45,5 @@
               <noise type="gaussian">
                 <mean>0.0</mean>
-                <stddev>0.009</stddev>
+                <stddev>0.000617</stddev>  <!-- ISM330DHCX: 5 mdps/√Hz * √50 Hz, converted to rad/s -->
               </noise>
             </x>
@@ -51,5 +51,5 @@
               <noise type="gaussian">
                 <mean>0.0</mean>
-                <stddev>0.009</stddev>
+                <stddev>0.000617</stddev>
               </noise>
             </y>
@@ -57,5 +57,5 @@
               <noise type="gaussian">
                 <mean>0.0</mean>
-                <stddev>0.009</stddev>
+                <stddev>0.000617</stddev>
               </noise>
             </z>
@@ -65,5 +65,5 @@
               <noise type="gaussian">
                 <mean>0.0</mean>
-                <stddev>0.021</stddev>
+                <stddev>0.004162</stddev>  <!-- ISM330DHCX: 60 µg/√Hz * √50 Hz, converted to m/s² -->
               </noise>
             </x>
@@ -71,5 +71,5 @@
               <noise type="gaussian">
                 <mean>0.0</mean>
-                <stddev>0.021</stddev>
+                <stddev>0.004162</stddev>
               </noise>
             </y>
@@ -77,5 +77,5 @@
               <noise type="gaussian">
                 <mean>0.0</mean>
-                <stddev>0.021</stddev>
+                <stddev>0.004162</stddev>
               </noise>
             </z>

File: amiga_description/urdf/amiga_lidar.urdf.xacro (robot description, xacro)
@@ -1,7 +1,8 @@
 <?xml version="1.0"?>
-<robot xmlns:xacro="http://ros.org">
+<robot xmlns:xacro="http://www.ros.org/wiki/xacro">
   <xacro:macro name="lidar" params="prefix lidar_name parent_link">
     <xacro:property name="lidar_mass" value="1.0"/>
     <xacro:property name="lidar_xyz" value="0.65 0 ${0.232/2}"/>
+    <!-- <xacro:property name='lidar_xyz' value='0.65 0 ${0.4}'/> -->
     <xacro:property name="lidar_rpy" value="0 0 0"/>
     <link name="${prefix}__${lidar_name}">
@@ -40,5 +41,5 @@
           <scan>
             <horizontal>
-              <samples>360</samples>
+              <samples>1080</samples> <!-- 1080 samples for 0.33 degree resolution over 360 degrees -->
               <resolution>1</resolution>
               <min_angle>-1.57079632679</min_angle>
