Commit message: adding files for merge

File: amiga_description/urdf/amiga_body.urdf.xacro (robot description, xacro)
@@ -23,5 +23,5 @@
         <origin rpy="0.0 0.0 0.0" xyz="0.0 0.0 0.0"/>
         <geometry>
-          <mesh filename="file://$(find amiga_description)/meshes/farm-ng/amiga/frame_on_amiga_v2_simplified.stl"/>
+          <mesh filename="file://$(find amiga_description)/meshes/frame_on_amiga_v2_simplified.stl"/>
         </geometry>
         <material name="LightLightGrey"/>

File: amiga_description/urdf/amiga_ros2_control.urdf.xacro (robot description, xacro)
@@ -24,8 +24,26 @@
         </xacro:unless>
       </hardware>
-      <joint name="${prefix}linear_slider_joint">
-        <command_interface name="position"/>
+      <joint name="${prefix}__left_wheel_front_joint">
+        <command_interface name="velocity"/>
+        <state_interface name="velocity"/>
         <state_interface name="position"/>
+        <state_interface name="effort"/>
+      </joint>
+      <joint name="${prefix}__right_wheel_front_joint">
+        <command_interface name="velocity"/>
         <state_interface name="velocity"/>
+        <state_interface name="position"/>
+        <state_interface name="effort"/>
+      </joint>
+      <joint name="${prefix}__left_wheel_rear_joint">
+        <command_interface name="velocity"/>
+        <state_interface name="velocity"/>
+        <state_interface name="position"/>
+        <state_interface name="effort"/>
+      </joint>
+      <joint name="${prefix}__right_wheel_rear_joint">
+        <command_interface name="velocity"/>
+        <state_interface name="velocity"/>
+        <state_interface name="position"/>
         <state_interface name="effort"/>
       </joint>

Commit message: Odom now matches what the robot is actually doing lol

File: amiga_description/urdf/amiga_body.urdf.xacro (robot description, xacro)
@@ -21,5 +21,5 @@
     <link name="${prefix}__body">
       <visual>
-        <origin rpy="0.0 0.0 0.0" xyz="0.0 0.0 0.0"/>
+        <origin rpy="0.0 0.0 3.14159265359" xyz="0.0 0.0 0.0"/>
         <geometry>
           <mesh filename="file://$(find amiga_description)/meshes/frame_on_amiga_v2_simplified.stl"/>
@@ -46,5 +46,5 @@
       </collision> -->
       <inertial>
-        <origin rpy="0 0 0" xyz="0.0 0.0 0.0"/>
+        <origin rpy="0 0 3.14159265359" xyz="0.0 0.0 0.0"/>
         <mass value="${amiga_mass}"/>
         <inertia ixx="${1/12 * amiga_mass * (amiga_collision_box0_y**2 + amiga_collision_box0_z**2)}"

File: amiga_description/urdf/amiga_lidar.urdf.xacro (robot description, xacro)
@@ -3,6 +3,6 @@
   <xacro:macro name="lidar" params="prefix lidar_name parent_link">
     <xacro:property name="lidar_mass" value="1.0"/>
-    <xacro:property name="lidar_xyz" value="-0.65 0 ${0.232/2}"/>
-    <xacro:property name="lidar_rpy" value="0 0 3.14159265359"/>
+    <xacro:property name="lidar_xyz" value="0.65 0 ${0.232/2}"/>
+    <xacro:property name="lidar_rpy" value="0 0 0"/>
     <link name="${prefix}__${lidar_name}">
       <visual>

File: amiga_description/urdf/amiga_macro.urdf.xacro (robot description, xacro)
@@ -35,7 +35,7 @@
     wheel_name="right_wheel_rear"
     parent_link="${amiga_prefix}__base"
-    joint_origin_xyz="0.344 0.5 0.22"
+    joint_origin_xyz="-0.344 -0.5 0.22"
     joint_origin_rpy="0 0 0"
-    joint_axis_xyz="0 -1 0"
+    joint_axis_xyz="0 1 0"
     wheel_radius="${wheel_radius}"
     wheel_width="${wheel_width}"
@@ -46,7 +46,7 @@
     wheel_name="left_wheel_rear"
     parent_link="${amiga_prefix}__base"
-    joint_origin_xyz="0.344 -0.5 0.22"
+    joint_origin_xyz="-0.344 0.5 0.22"
     joint_origin_rpy="0 0 0"
-    joint_axis_xyz="0 -1 0"
+    joint_axis_xyz="0 1 0"
     wheel_radius="${wheel_radius}"
     wheel_width="${wheel_width}"
@@ -57,7 +57,7 @@
     wheel_name="right_wheel_front"
     parent_link="${amiga_prefix}__base"
-    joint_origin_xyz="-0.344 0.5 0.22"
+    joint_origin_xyz="0.344 -0.5 0.22"
     joint_origin_rpy="0 0 0"
-    joint_axis_xyz="0 -1 0"
+    joint_axis_xyz="0 1 0"
     wheel_radius="${wheel_radius}"
     wheel_width="${wheel_width}"
@@ -68,7 +68,7 @@
     wheel_name="left_wheel_front"
     parent_link="${amiga_prefix}__base"
-    joint_origin_xyz="-0.344 -0.5 0.22"
+    joint_origin_xyz="0.344 0.5 0.22"
     joint_origin_rpy="0 0 0"
-    joint_axis_xyz="0 -1 0"
+    joint_axis_xyz="0 1 0"
     wheel_radius="${wheel_radius}"
     wheel_width="${wheel_width}"

File: amiga_description/urdf/amiga_wheel.urdf.xacro (robot description, xacro)
@@ -17,5 +17,5 @@
       </collision>
       <inertial>
-        <origin xyz="0 0 0" rpy="0 0 0"/>
+        <origin xyz="0 0 0" rpy="1.5708 0 0"/>
         <mass value="${wheel_mass}"/>
         <inertia

Commit message: moved IMU to be along axis of rotation to fix EKF issues

File: amiga_description/urdf/amiga_body.urdf.xacro (robot description, xacro)
@@ -5,5 +5,5 @@
       <color rgba="0.941 0.941 0.941 1.0"/>
     </material>
-    <xacro:property name="amiga_mass" value="40.0"/>
+    <xacro:property name="amiga_mass" value="140.0"/>
     <xacro:property name="amiga_collision_box0_x" value='1.132'/>
     <xacro:property name="amiga_collision_box0_y" value='0.800'/>

File: amiga_description/urdf/amiga_imu.urdf.xacro (robot description, xacro)
@@ -3,5 +3,5 @@
   <xacro:macro name="imu" params="prefix imu_name parent_link">
     <xacro:property name="imu_mass" value="0.1"/>
-    <xacro:property name="imu_xyz" value="0 0.1 0.8"/>
+    <xacro:property name="imu_xyz" value="0 0.0 0.8"/>
     <xacro:property name="imu_rpy" value="0 0 0"/>
     <link name="${prefix}__${imu_name}">

File: amiga_description/urdf/amiga_lidar.urdf.xacro (robot description, xacro)
@@ -3,6 +3,6 @@
   <xacro:macro name="lidar" params="prefix lidar_name parent_link">
     <xacro:property name="lidar_mass" value="1.0"/>
-    <xacro:property name="lidar_xyz" value="0.65 0 ${0.232/2}"/>
-    <!-- <xacro:property name='lidar_xyz' value='0.65 0 ${0.4}'/> -->
+    <!-- <xacro:property name="lidar_xyz" value="0.65 0 ${0.232/2}"/> -->
+    <xacro:property name='lidar_xyz' value='0.65 0 1.6'/>
     <xacro:property name="lidar_rpy" value="0 0 0"/>
     <link name="${prefix}__${lidar_name}">
@@ -43,6 +43,6 @@
               <samples>1080</samples> <!-- 1080 samples for 0.33 degree resolution over 360 degrees -->
               <resolution>1</resolution>
-              <min_angle>-1.57079632679</min_angle>
-              <max_angle>1.57079632679</max_angle>
+              <min_angle>-${pi}</min_angle>
+              <max_angle>${pi}</max_angle>
             </horizontal>
           </scan>

File: amiga_description/urdf/amiga_wheel.urdf.xacro (robot description, xacro)
@@ -36,5 +36,6 @@
     <gazebo reference="${prefix}__${wheel_name}">
       <mu1>1.0</mu1> <!-- longitudinal friction (rolling direction) -->
-      <mu2>0.5</mu2> <!-- lateral friction (sideways direction) -->
+      <!-- <mu2>0.5</mu2> lateral friction (sideways direction) -->
+       <mu2>0.1</mu2>
       <fdir1>1 0 0</fdir1> <!-- friction direction -->
     </gazebo>
